Commit message: Twin bake + Estun read-only mirror: J5 axis fix, high-res navy geometry, URDF deploy, dashboard control surface (joint sliders, 6-DOF IK gizmo, coordinated Home), render-stability fix, estun_driver telemetry (monitor_only), DH fit checkpoint
Co-Authored-By: Claude Opus 4.7 <noreply@anthropic.com>

File: models/robots/estun_s10-140/s10-140-provisional.urdf (robot description, URDF)
Before this commit: robot estun_s10_140_provisional, 9 links, 8 joints
Joints:
- removed joint J1
- removed joint J2
- removed joint J3
- removed joint J4
- removed joint J5
- removed joint J6
- added joint joint_1: type revolute, parent base_link, child link1_shoulder, origin xyz=0 0 0.186 rpy=0 0 0, axis 0 0 1, limit lower=-6.2832 upper=6.2832 effort=150 velocity=2.6180
- added joint joint_2: type revolute, parent link1_shoulder, child link2_upper_arm, origin xyz=0 0.221 0 rpy=0 0 0, axis 0 1 0, limit lower=-6.2832 upper=6.2832 effort=150 velocity=2.6180
- added joint joint_3: type revolute, parent link2_upper_arm, child link3_forearm, origin xyz=0 0 0.700 rpy=0 0 0, axis 0 1 0, limit lower=-2.7925 upper=2.7925 effort=150 velocity=2.6180
- added joint joint_4: type revolute, parent link3_forearm, child link4_wrist1, origin xyz=0 0.175 0.700 rpy=0 0 0, axis 0 0 1, limit lower=-6.2832 upper=6.2832 effort=50 velocity=3.1416
- added joint joint_5: type revolute, parent link4_wrist1, child link5_wrist2, origin xyz=0 0 0.1615 rpy=0 0 0, axis 0 1 0, limit lower=-6.2832 upper=6.2832 effort=50 velocity=3.1416
- added joint joint_6: type revolute, parent link5_wrist2, child link6_flange, origin xyz=0 0 0.1505 rpy=0 0 0, axis 0 0 1, limit lower=-6.2832 upper=6.2832 effort=50 velocity=3.1416
